Commit message: update

File: kortex_description/robots/gen3_robotiq_2f_85.xacro (robot description, xacro)
@@ -1,4 +1,5 @@
 <?xml version="1.0"?>
 <robot name="gen3_robotiq_2f_85" xmlns:xacro="http://ros.org/wiki/xacro">
+    <!-- <robot xmlns:xacro="http://ros.org/wiki/xacro"> -->
     <!-- Arguments -->
     <xacro:arg name="arm" default="gen3" />
@@ -6,5 +7,5 @@
     <xacro:arg name="vision" default="true" />
     <xacro:arg name="gripper" default="robotiq_2f_85" />
-    <xacro:arg name="sim" default="false" />
+    <xacro:arg name="sim" default="true" />
     <xacro:arg name="prefix" default="" />
     <xacro:include filename="$(find kortex_description)/robots/kortex_robot.xacro" />

File: kortex_description/robots/kortex_robot.xacro (robot description, xacro)
@@ -7,4 +7,5 @@
             <xacro:include filename="$(find kortex_description)/grippers/${gripper}/urdf/${gripper}_macro.xacro" />
         </xacro:unless>
+        <xacro:include filename="$(find kortex_description)/base/urdf/base_macro.xacro" />
         <xacro:if value="${sim}">
             <!-- Arm transmission elements-->
@@ -17,5 +18,5 @@
         <!-- Run the macros -->
         <!-- For gazebo-->
-        <xacro:if value="${sim}">
+        <!-- <xacro:if value="${sim}">
             <link name="world" />
             <joint name="world_to_root" type="fixed">
@@ -24,5 +25,14 @@
                 <origin xyz="0 0 0" rpy="0 0 0" />
             </joint>
+        </xacro:if> -->
+        <xacro:if value="${sim}">
+            <joint name="arm_to_mobile_base" type="fixed">
+                <child link="${prefix}base_link" />
+                <parent link="base_link" />
+                <origin xyz="0 0 0.184" rpy="0 0 0" />
+            </joint>
         </xacro:if>
+        <!-- Load the base -->
+        <xacro:load_base />
         <!-- Load the arm -->
         <xacro:load_arm parent="" dof="${dof}" vision="${vision}" prefix="${prefix}">
