Commit message: mobile base update

File: kortex_description/grippers/robotiq_2f_85/urdf/robotiq_2f_85_transmission_macro.xacro (robot description, xacro)
@@ -4,5 +4,5 @@
         <transmission name="finger_joint_trans">
             <type>transmission_interface/SimpleTransmission</type>
-            <joint name="finger_joint">
+            <joint name="${prefix}finger_joint">
                 <hardwareInterface>hardware_interface/PositionJointInterface</hardwareInterface>
             </joint>
@@ -14,5 +14,5 @@
         <gazebo>
             <plugin filename="libroboticsgroup_gazebo_mimic_joint_plugin.so" name="mimic_robotiq_85_1">
-                <joint>finger_joint</joint>
+                <joint>${prefix}finger_joint</joint>
                 <mimicJoint>right_outer_knuckle_joint</mimicJoint>
                 <multiplier>1.0</multiplier>
@@ -21,5 +21,5 @@
             </plugin>
             <plugin filename="libroboticsgroup_gazebo_mimic_joint_plugin.so" name="mimic_robotiq_85_2">
-                <joint>finger_joint</joint>
+                <joint>${prefix}finger_joint</joint>
                 <mimicJoint>right_inner_knuckle_joint</mimicJoint>
                 <multiplier>1.0</multiplier>
@@ -28,5 +28,5 @@
             </plugin>
             <plugin filename="libroboticsgroup_gazebo_mimic_joint_plugin.so" name="mimic_robotiq_85_3">
-                <joint>finger_joint</joint>
+                <joint>${prefix}finger_joint</joint>
                 <mimicJoint>left_inner_knuckle_joint</mimicJoint>
                 <multiplier>1.0</multiplier>
@@ -35,5 +35,5 @@
             </plugin>
             <plugin filename="libroboticsgroup_gazebo_mimic_joint_plugin.so" name="mimic_robotiq_85_4">
-                <joint>finger_joint</joint>
+                <joint>${prefix}finger_joint</joint>
                 <mimicJoint>left_inner_finger_joint</mimicJoint>
                 <multiplier>-1.0</multiplier>
@@ -42,5 +42,5 @@
             </plugin>
             <plugin filename="libroboticsgroup_gazebo_mimic_joint_plugin.so" name="mimic_robotiq_85_5">
-                <joint>finger_joint</joint>
+                <joint>${prefix}finger_joint</joint>
                 <mimicJoint>right_inner_finger_joint</mimicJoint>
                 <multiplier>-1.0</multiplier>

File: kortex_description/robots/gen3_robotiq_2f_85.xacro (robot description, xacro)
@@ -8,5 +8,5 @@
     <xacro:arg name="gripper" default="robotiq_2f_85" />
     <xacro:arg name="sim" default="true" />
-    <xacro:arg name="prefix" default="" />
+    <xacro:arg name="prefix" default="arm_" />
     <xacro:include filename="$(find kortex_description)/robots/kortex_robot.xacro" />
     <xacro:load_robot arm="$(arg arm)" gripper="$(arg gripper)" dof="$(arg dof)" vision="$(arg vision)" sim="$(arg sim)" prefix="$(arg prefix)" />

File: kortex_description/robots/kortex_robot.xacro (robot description, xacro)
@@ -7,5 +7,6 @@
             <xacro:include filename="$(find kortex_description)/grippers/${gripper}/urdf/${gripper}_macro.xacro" />
         </xacro:unless>
-        <xacro:include filename="$(find kortex_description)/base/urdf/base_macro.xacro" />
+        <!-- <xacro:include filename="$(find kortex_description)/base/urdf/base_macro.xacro" /> -->
+        <xacro:include filename="$(find kortex_description)/base/urdf/freight_macro.xacro" />
         <xacro:if value="${sim}">
             <!-- Arm transmission elements-->
@@ -29,6 +30,6 @@
             <joint name="arm_to_mobile_base" type="fixed">
                 <child link="${prefix}base_link" />
-                <parent link="base_link" />
-                <origin xyz="0 0 0.184" rpy="0 0 0" />
+                <parent link="chassis_link" />
+                <origin xyz="0 0 0.36" rpy="0 0 0" />
             </joint>
         </xacro:if>
