Commit message: update

File: kortex_description/base/urdf/freight_macro.xacro (robot description, xacro)
@@ -2,5 +2,6 @@
 <robot name="freight" xmlns:xacro="http://www.ros.org/wiki/xacro">
   <xacro:macro name="load_base" >
-      <xacro:include filename="$(find fetch_description)/robots/freight.urdf" />
+      <!-- <xacro:include filename="$(find fetch_description)/robots/freight.urdf.xacro" /> -->
+      <xacro:include filename="$(find kortex_description)/base/urdf/freight.urdf.xacro" />
       <!-- Base is modeled as a big tub sitting on floor, with two wheels -->
       <gazebo reference="chassis_link">
@@ -39,9 +40,13 @@
         <implicitSpringDamper>1</implicitSpringDamper>
       </gazebo>
+      <gazebo reference="camera_support">
+        <material>Gazebo/Black</material>
+      </gazebo>
       <!-- SICK TIM561 (25m Range) -->
-      <gazebo reference="laser_link">
+      <gazebo reference="${ns}/laser_link">
+      <!-- <gazebo reference="laser_link">   <! TEMPORARY FIX -->
         <sensor type="ray" name="base_laser">
           <pose>0 0 0 0 0 0</pose>
-          <visualize>true</visualize>
+          <visualize>false</visualize>
           <update_rate>15</update_rate>
           <ray>

File: kortex_description/robots/gen3_robotiq_2f_85.xacro (robot description, xacro)
@@ -9,5 +9,6 @@
     <xacro:arg name="sim" default="true" />
     <xacro:arg name="prefix" default="arm_" />
+    <xacro:arg name="ns" default="my_$(arg arm)" />
     <xacro:include filename="$(find kortex_description)/robots/kortex_robot.xacro" />
-    <xacro:load_robot arm="$(arg arm)" gripper="$(arg gripper)" dof="$(arg dof)" vision="$(arg vision)" sim="$(arg sim)" prefix="$(arg prefix)" />
+    <xacro:load_robot arm="$(arg arm)" gripper="$(arg gripper)" dof="$(arg dof)" vision="$(arg vision)" sim="$(arg sim)" prefix="$(arg prefix)" ns="$(arg ns)" />
 </robot>

File: kortex_description/robots/kortex_robot.xacro (robot description, xacro)
@@ -1,5 +1,5 @@
 <?xml version="1.0"?>
 <robot xmlns:xacro="http://ros.org/wiki/xacro">
-    <xacro:macro name="load_robot" params="arm gripper dof vision sim prefix">
+    <xacro:macro name="load_robot" params="arm gripper dof vision sim prefix ns">
         <!-- Files to include -->
         <xacro:include filename="$(find kortex_description)/arms/${arm}/${dof}dof/urdf/${arm}_macro.xacro" />
@@ -31,5 +31,5 @@
                 <child link="${prefix}base_link" />
                 <parent link="chassis_link" />
-                <origin xyz="0 0 0.36" rpy="0 0 0" />
+                <origin xyz="0.1 0 0.36" rpy="0 0 0" />
             </joint>
         </xacro:if>
